File: pcb-main.brd (EAGLE design)
At the start: 100 x 80 mm, 22 parts, among them U1 BTA-RX-A, U2 RS3-1205S

Commit message: Component rename
Parts:
- R3: value 2.2R -> 2R2(TH)
Changed lines of the file:
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@@
 <attribute name="MOUSER" value="81-BL01RN1A1F1J" x="-0.5" y="74" size="1.778" layer="27" display="off"/>
 </element>
-<element name="R3" library="resistors" package="R-0207/10" value="2.2R" x="31.5" y="44" rot="R270"/>
+<element name="R3" library="resistors" package="R-0207/10" value="2R2(TH)" x="31.5" y="44" rot="R270"/>
 <element name="C1" library="capacitors" package="C050-024X044" value="100N(TH)" x="7" y="52.5" rot="R90">
 <attribute name="MOUSER" value="81-RCER71H104K0A2H3B" x="7" y="52.5" size="1.778" layer="27" rot="R90" display="off"/>

Commit message: Change DC Connector
Parts:
- XS1: value 712RA -> 722RA
Other:
- outline, holes or cut-outs redrawn
Changed lines of the file:
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@@
 <wire x1="0" y1="2" x2="0" y2="78" width="0" layer="20"/>
 <wire x1="0" y1="78" x2="2" y2="80" width="0" layer="20" curve="-90"/>
-<wire x1="2" y1="80" x2="98" y2="80" width="0" layer="20"/>
+<wire x1="2" y1="80" x2="98" y2="80" width="0" layer="21"/>
 <wire x1="98" y1="80" x2="100" y2="78" width="0" layer="20" curve="-90"/>
 <wire x1="100" y1="78" x2="100" y2="2" width="0" layer="20"/>
@@
 <wire x1="2" y1="0" x2="46.5" y2="0" width="0" layer="20"/>
 <wire x1="53.5" y1="0" x2="98" y2="0" width="0" layer="20"/>
-<wire x1="44" y1="79" x2="44" y2="77" width="0.254" layer="20"/>
-<wire x1="44" y1="77" x2="53" y2="77" width="0.254" layer="20"/>
-<wire x1="53" y1="77" x2="53" y2="79" width="0.254" layer="20"/>
-<wire x1="53" y1="79" x2="44" y2="79" width="0.254" layer="20"/>
+<wire x1="44" y1="79" x2="44" y2="77" width="0.254" layer="21"/>
+<wire x1="44" y1="77" x2="53" y2="77" width="0.254" layer="21"/>
+<wire x1="53" y1="77" x2="53" y2="79" width="0.254" layer="21"/>
+<wire x1="53" y1="79" x2="44" y2="79" width="0.254" layer="21"/>
 <wire x1="46.5" y1="0" x2="47.5" y2="1" width="0" layer="20" curve="-90"/>
 <wire x1="47.5" y1="1" x2="52.5" y2="1" width="0" layer="20"/>
@@
 <attribute name="MOUSER" value="71-RN55D-F-1.0K" x="37" y="28.5" size="1.778" layer="27" rot="R180" display="off"/>
 </element>
-<element name="XS1" library="connectors" package="SWITCHCRAFT-L712RA" value="712RA" x="10" y="80" rot="R270">
+<element name="XS1" library="connectors" package="SWITCHCRAFT-L712RA" value="722RA" x="10" y="80" rot="R270">
 <attribute name="MOUSER" value="502-722RA" x="23.5" y="93" size="1.778" layer="27" rot="R270" display="off"/>
 </element>
