File: pcb-main.sch (EAGLE design)
At the start: 21 parts, among them U1 BTA-RX-A, U2 RS3-1205S

Commit message: Component rename
Parts:
- R3: value 2.2R -> 2R2(TH); device resistors:R-0207/10 -> resistors:2R2(TH)
Changed lines of the file:
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@@
 <part name="GND5" library="supply" deviceset="CHASSIS" device=""/>
 <part name="GND3" library="supply" deviceset="CHASSIS" device=""/>
-<part name="R3" library="resistors" deviceset="R" device="-0207/10" value="2.2R"/>
+<part name="R3" library="resistors" deviceset="?" device="2R2(TH)" value="2R2(TH)"/>
 <part name="GND2" library="supply" deviceset="CHASSIS" device=""/>
 <part name="GND7" library="supply" deviceset="GND" device=""/>

Commit message: Change DC Connector
Parts:
- XS1: value 712RA -> 722RA; device connectors:712RA -> connectors:722RA
Changed lines of the file:
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@@
 <part name="PWR2" library="supply" deviceset="+5V" device=""/>
 <part name="PWR1" library="supply" deviceset="+5V" device=""/>
-<part name="XS1" library="connectors" deviceset="712RA" device=""/>
+<part name="XS1" library="connectors" deviceset="722RA" device=""/>
 <part name="GND1" library="supply" deviceset="CHASSIS" device=""/>
 <part name="VD1" library="diodes-schottky" deviceset="?" device="STPS2L60"/>

Commit message: Swap Prev/Next Buttons
Connections:
- removed net N$39: SB2.1.CM, U1.3
- removed net N$40: SB3.1.CM, U1.4
- new net N$1: SB2.1.CM, U1.4
- new net N$2: SB3.1.CM, U1.3
Changed lines of the file:
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@@
-</segment>
-</net>
-<net name="N$39" class="0">
-<segment>
-<pinref part="U1" gate="G$1" pin="3"/>
-<wire x1="-17.78" y1="-10.16" x2="-17.78" y2="-25.4" width="0.1524" layer="91"/>
-<pinref part="SB2" gate=".1" pin="CM"/>
-<wire x1="-17.78" y1="-25.4" x2="-25.4" y2="-25.4" width="0.1524" layer="91"/>
-</segment>
-</net>
-<net name="N$40" class="0">
-<segment>
-<pinref part="U1" gate="G$1" pin="4"/>
-<wire x1="-12.7" y1="-10.16" x2="-12.7" y2="-33.02" width="0.1524" layer="91"/>
-<pinref part="SB3" gate=".1" pin="CM"/>
-<wire x1="-12.7" y1="-33.02" x2="-25.4" y2="-33.02" width="0.1524" layer="91"/>
 </segment>
 </net>
@@
 </segment>
 </net>
+<net name="N$1" class="0">
+<segment>
+<pinref part="SB2" gate=".1" pin="CM"/>
+<pinref part="U1" gate="G$1" pin="4"/>
+<wire x1="-25.4" y1="-25.4" x2="-12.7" y2="-25.4" width="0.1524" layer="91"/>
+<wire x1="-12.7" y1="-25.4" x2="-12.7" y2="-10.16" width="0.1524" layer="91"/>
+</segment>
+</net>
+<net name="N$2" class="0">
+<segment>
+<pinref part="SB3" gate=".1" pin="CM"/>
+<pinref part="U1" gate="G$1" pin="3"/>
+<wire x1="-25.4" y1="-33.02" x2="-17.78" y2="-33.02" width="0.1524" layer="91"/>
+<wire x1="-17.78" y1="-33.02" x2="-17.78" y2="-10.16" width="0.1524" layer="91"/>
+</segment>
+</net>

Commit message: Bump board revision
Parts:
- PCB1: value IO-BT rev.A -> IO-BT rev.B
Changed lines of the file:
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@@
 <parts>
 <part name="O1" library="hardware" deviceset="MOUNT(?)" device="KEYSTONE-7762"/>
-<part name="PCB1" library="module-footprints" deviceset="GENERIC" device="-LOGO" value="IO-BT rev.A"/>
+<part name="PCB1" library="module-footprints" deviceset="GENERIC" device="-LOGO" value="IO-BT rev.B"/>
 <part name="XS2" library="connectors" deviceset="ACJS-MHR" device=""/>
 <part name="XS3" library="connectors" deviceset="ACJS-MHR" device=""/>
