File: pcb-main.sch (EAGLE design)
At the start: 21 parts, among them U1 BTA-RX-A, U2 RS3-1205S

Commit message: Updates
- Added output volume potentiometer
- Blue LED is now used for signal indicator
- Removed next/prev buttons
Parts:
- removed O1: MOUNT(KEYSTONE-7762), hardware:MOUNT(KEYSTONE-7762)
- removed SB2, SB3: SPUN191000, switches:SPUN191000
- added C10, C11: 22P(TH), capacitors:22P(TH)
- added C6, C7: 470U/35V, capacitors-electrolytic:470U/35V
- added C8, C9: 100N(TH), capacitors:100N(TH)
- added DA1: NJM2068D, ic-jrc:NJM2068D
- added R10, R11: 100R(TH), resistors:100R(TH)
- added R12, R13: 100K(TH), resistors:100K(TH)
- added R4: 2R2(TH), resistors:2R2(TH)
- added R5: 2A10K(PTD90), potentiometers:2A10K(PTD90)
- added R6, R7, R8, R9: 10K(TH), resistors:10K(TH)
- added VD2: 1N4148, diodes:1N4148
- added VT1: BC548, transistors-npn:BC548
- R1, R2: value 1K(TH) -> 1K5(TH); device resistors:1K(TH) -> resistors:1K5(TH)
- U2: value RS3-1205S -> RS3-1205D; device regulators-switch-mode:RS3-1205S -> regulators-switch-mode:RS3-1205D
Connections:
- removed net N$35: U1.12, XS2.R, XS2.S, XS3.R, XS3.S
- removed net N$36: U1.10, XS2.T
- removed net N$37: U1.11, XS3.T
- removed net N$45: R2.2, U1.7
- new net -5V: C7.-, C9.1, DA1*.V-, R4.2
- new net N$10: R10.2, XS2.T
- new net N$11: R11.2, XS3.T
- new net N$12: R2.2, VT1.C
- new net N$13: R12.2, R13.2, VD2.C, VT1.B
- new net N$3: R5.2.W, R6.1
- new net N$4: C11.1, DA1.1.IN-, R6.2, R7.1
- new net N$5: C10.1, DA1.2.IN-, R8.2, R9.1
- new net N$6: R12.1, R5.1.CW, U1.10
- new net N$7: R13.1, R5.2.CW, U1.11
- new net N$8: C10.2, DA1.2.OUT, R10.1, R9.2
- new net N$9: C11.2, DA1.1.OUT, R11.1, R7.2
- net +5V: now also C8.2, DA1*.V+
- net GND: now also C6.+, C7.+, C8.1, C9.2, DA1.1.IN+, DA1.2.IN+, R5.1.CCW, R5.2.CCW, U1.12, U2.GND, VD2.A, VT1.E, XS2.R, XS2.S, XS3.R, XS3.S; no longer U2.V-
- net N$1: now also C6.-, R4.1, U2.V-; no longer SB2.1.CM, U1.4
- net N$2: now also R5.1.W, R8.1; no longer SB3.1.CM, U1.3
- net N$41: no longer SB2.1.NO, SB3.1.NO
Other:
- moved on the sheet: C4, C5, R3, XS2, XS3
